File: templates/Projects/mikroBUS-M/mikroBUS-M.kicad_pcb (KiCad board)
At the start: 2 copper layers, 25.4 x 42.9 mm, 4 parts, among them CON101 MIKROBUS_MODULE_CONN

Commit message: Upgrade mikroBUS templates to v8.
Other:
- net class Default removed
